File: HS Numpad/HS Numpad.kicad_sch (KiCad schematic)
At the start: 44 parts, among them J1 Conn_01x05_MountingPin, U1 Nice_Nano_V2

Commit message: update
Parts:
- J1: footprint (none) -> Connector_PinHeader_2.54mm:PinHeader_1x05_P2.54mm_Vertical
Connections:
- net CS: now also U1.1; no longer U1.13 (10)
- net GND: now also U1.3 (GND); no longer U1.22 (RST)
- net MOSI: now also U1.14 (16), U1.5 (2); no longer U1.11 (8)
- net ROW0: now also U1.8 (5); no longer U1.5 (2)
- net ROW1: now also U1.9 (6); no longer U1.6 (3)
- net ROW2: now also U1.10 (7); no longer U1.7 (4)
- net ROW3: now also U1.11 (8); no longer U1.8 (5)
- net SCK: now also U1.16 (15), U1.6 (3); no longer U1.9 (6)
- net VCC: now also U1.21 (3.3v); no longer U1.4 (GND)
Other:
- moved on the sheet: MX20, MX21, U1
